File: Dual LPF/Dual LPF V1.2 Bottom.brd (EAGLE design)
At the start: 55 x 87 mm, 48 parts, among them IC2 TL074, IC3 V2164, IC4 TL074

Commit message: Add files via upload
Minor resistor value change
Parts:
- FILM_C1, FILM_C2, FILM_C3, FILM_C4: value 470nF -> 1uF
- R20, R21, R23, R27, R32, R33, R35, R39: value 33k -> 30k
Other:
- board text added: "Main Board Dual Dreadful VCF V1.3 Tom Evans 2019 CC BY 4.0"
- board text removed: "Main Board Dual Dreadful VCF V1.2 Tom Evans 2019 Design based on Dreadbox Erebus"
