File: Dual LPF/Dual LPF V1.2 Top.brd (EAGLE design)
At the start: 60 x 100 mm, 36 parts, among them U3 TL074_

Commit message: Add files via upload
Minor resistor value change
Other:
- board text added: "Control Board Dual Dreadful VCF V1.2 Tom Evans 2019 CC BY 4.0"
- board text removed: "Control Board Dual Dreadful VCF V1.2 Tom Evans 2019 Design based on Dreadbox Erebus"
Changed lines of the file:
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@@
 <?xml version="1.0" encoding="utf-8"?>
 <!DOCTYPE eagle SYSTEM "eagle.dtd">
-<eagle version="9.0.0">
+<eagle version="9.3.0">
 <drawing>
 <settings>
@@
 Dual Dreadful VCF V1.2
 Tom Evans 2019
-Design based on Dreadbox Erebus</text>
+CC BY 4.0</text>
 <hole x="55" y="92" drill="3.2"/>
 </plain>
@@
 <param name="checkStop" value="0"/>
 <param name="checkValues" value="0"/>
+<param name="checkNames" value="1"/>
+<param name="checkWireStubs" value="1"/>
+<param name="checkPolygonWidth" value="0"/>
 <param name="useDiameter" value="13"/>
 <param name="maxErrors" value="50"/>
@@
 </autorouter>
 <elements>
-<element name="CUTOFF1" library="MusicThingModular" package="9MM_SNAP-IN_POT" value="B100k" x="44" y="87"/>
-<element name="CUTOFF2" library="MusicThingModular" package="9MM_SNAP-IN_POT" value="B100k" x="44" y="44"/>
-<element name="FCV1" library="MusicThingModular" package="WQP-PJ301M-12_JACK" value="THONKICONNNEW" x="13" y="17" rot="R180"/>
-<element name="FCV1_AMT" library="MusicThingModular" package="9MM_SNAP-IN_POT" value="B100k" x="11" y="77"/>
-<element name="FCV2_AMT" library="MusicThingModular" package="9MM_SNAP-IN_POT" value="B100k" x="11" y="34"/>
-<element name="FCV2" library="MusicThingModular" package="WQP-PJ301M-12_JACK" value="THONKICONNNEW" x="30" y="17" rot="R180"/>
-<element name="IN1" library="MusicThingModular" package="WQP-PJ301M-12_JACK" value="THONKICONNNEW" x="7" y="5" rot="R90"/>
-<element name="IN2" library="MusicThingModular" package="WQP-PJ301M-12_JACK" value="THONKICONNNEW" x="21" y="5" rot="R90"/>
-<element name="OUT1" library="MusicThingModular" package="WQP-PJ301M-12_JACK" value="THONKICONNNEW" x="39" y="5" rot="R270"/>
-<element name="OUT2" library="MusicThingModular" package="WQP-PJ301M-12_JACK" value="THONKICONNNEW" x="53" y="5" rot="R270"/>
+<element name="CUTOFF1" library="MusicThingModular" package="9MM_SNAP-IN_POT" value="B100k" x="44" y="87" smashed="yes">
+<attribute name="NAME" x="40.19" y="89.54" size="1.0668" layer="25"/>
+<attribute name="VALUE" x="40.19" y="83.19" size="1.27" layer="27"/>
+</element>
+<element name="CUTOFF2" library="MusicThingModular" package="9MM_SNAP-IN_POT" value="B100k" x="44" y="44" smashed="yes">
+<attribute name="NAME" x="40.19" y="46.54" size="1.0668" layer="25"/>
+<attribute name="VALUE" x="40.19" y="40.19" size="1.27" layer="27"/>
+</element>
+<element name="FCV1" library="MusicThingModular" package="WQP-PJ301M-12_JACK" value="THONKICONNNEW" x="13" y="17" smashed="yes" rot="R180">
+<attribute name="NAME" x="8.4788" y="21.7244" size="1.016" layer="21" rot="SR0"/>
+</element>
+<element name="FCV1_AMT" library="MusicThingModular" package="9MM_SNAP-IN_POT" value="B100k" x="11" y="77" smashed="yes">
+<attribute name="NAME" x="7.19" y="79.54" size="1.0668" layer="25"/>
+<attribute name="VALUE" x="7.19" y="73.19" size="1.27" layer="27"/>
+</element>
+<element name="FCV2_AMT" library="MusicThingModular" package="9MM_SNAP-IN_POT" value="B100k" x="11" y="34" smashed="yes">
+<attribute name="NAME" x="7.19" y="36.54" size="1.0668" layer="25"/>
+<attribute name="VALUE" x="7.19" y="30.19" size="1.27" layer="27"/>
+</element>
+<element name="FCV2" library="MusicThingModular" package="WQP-PJ301M-12_JACK" value="THONKICONNNEW" x="30" y="17" smashed="yes" rot="R180">
+<attribute name="NAME" x="25.4788" y="21.7244" size="1.016" layer="21" rot="SR0"/>
+</element>
+<element name="IN1" library="MusicThingModular" package="WQP-PJ301M-12_JACK" value="THONKICONNNEW" x="7" y="5" smashed="yes" rot="R90">
+<attribute name="NAME" x="11.7244" y="9.5212" size="1.016" layer="21" rot="SR270"/>
+</element>
+<element name="IN2" library="MusicThingModular" package="WQP-PJ301M-12_JACK" value="THONKICONNNEW" x="21" y="5" smashed="yes" rot="R90">
+<attribute name="NAME" x="25.7244" y="9.5212" size="1.016" layer="21" rot="SR270"/>
+</element>
+<element name="OUT1" library="MusicThingModular" package="WQP-PJ301M-12_JACK" value="THONKICONNNEW" x="39" y="5" smashed="yes" rot="R270">
+<attribute name="NAME" x="34.2756" y="0.4788" size="1.016" layer="21" rot="SR90"/>
+</element>
+<element name="OUT2" library="MusicThingModular" package="WQP-PJ301M-12_JACK" value="THONKICONNNEW" x="53" y="5" smashed="yes" rot="R270">
+<attribute name="NAME" x="48.2756" y="0.4788" size="1.016" layer="21" rot="SR90"/>
+</element>
 <element name="R1" library="resistor" library_urn="urn:adsk.eagle:library:348" package="0207/7" package3d_urn="urn:adsk.eagle:package:25942/1" value="100k" x="27.94" y="33.02" smashed="yes">
 <attribute name="VALUE" x="25.654" y="32.4612" size="1.27" layer="27" ratio="10"/>
@@
 <attribute name="VALUE" x="52.705" y="82.356159375" size="1.27" layer="27" ratio="10" rot="R90"/>
 </element>
-<element name="RES1" library="MusicThingModular" package="9MM_SNAP-IN_POT" value="B100k" x="11" y="95"/>
-<element name="RES2" library="MusicThingModular" package="9MM_SNAP-IN_POT" value="B100k" x="11" y="52"/>
-<element name="SPREAD" library="MusicThingModular" package="9MM_SNAP-IN_POT" value="B100k" x="27" y="64.5"/>
-<element name="SPREAD_CV" library="MusicThingModular" package="WQP-PJ301M-12_JACK" value="THONKICONNNEW" x="47" y="17" rot="R180"/>
-<element name="U3" library="MusicThingModular" package="DIL14" value="TL074_" x="41.91" y="63.5" rot="R270"/>
-<element name="TOP" library="pinhead" library_urn="urn:adsk.eagle:library:325" package="2X05" package3d_urn="urn:adsk.eagle:package:22470/2" value="" x="11.43" y="62.23"/>
-<element name="PWR_T" library="pinhead" library_urn="urn:adsk.eagle:library:325" package="2X03" package3d_urn="urn:adsk.eagle:package:22462/2" value="" x="46.99" y="29.21"/>
+<element name="RES1" library="MusicThingModular" package="9MM_SNAP-IN_POT" value="B100k" x="11" y="95" smashed="yes">
+<attribute name="NAME" x="7.19" y="97.54" size="1.0668" layer="25"/>
+<attribute name="VALUE" x="7.19" y="91.19" size="1.27" layer="27"/>
+</element>
+<element name="RES2" library="MusicThingModular" package="9MM_SNAP-IN_POT" value="B100k" x="11" y="52" smashed="yes">
+<attribute name="NAME" x="7.19" y="54.54" size="1.0668" layer="25"/>
+<attribute name="VALUE" x="7.19" y="48.19" size="1.27" layer="27"/>
+</element>
+<element name="SPREAD" library="MusicThingModular" package="9MM_SNAP-IN_POT" value="B100k" x="27" y="64.5" smashed="yes">
+<attribute name="NAME" x="23.19" y="67.04" size="1.0668" layer="25"/>
+<attribute name="VALUE" x="23.19" y="60.69" size="1.27" layer="27"/>
+</element>
+<element name="SPREAD_CV" library="MusicThingModular" package="WQP-PJ301M-12_JACK" value="THONKICONNNEW" x="47" y="17" smashed="yes" rot="R180">
+<attribute name="NAME" x="42.4788" y="21.7244" size="1.016" layer="21" rot="SR0"/>
+</element>
+<element name="U3" library="MusicThingModular" package="DIL14" value="TL074_" x="41.91" y="63.5" smashed="yes" rot="R270">
+<attribute name="NAME" x="41.889" y="55.445" size="1.016" layer="25" font="vector" ratio="10" align="center"/>
+<attribute name="VALUE" x="41.929" y="63.515" size="2.032" layer="27" font="vector" ratio="12" rot="R270" align="center"/>
+</element>
+<element name="TOP" library="pinhead" library_urn="urn:adsk.eagle:library:325" package="2X05" package3d_urn="urn:adsk.eagle:package:22470/2" value="" x="11.43" y="62.23" smashed="yes">
+<attribute name="NAME" x="5.08" y="65.405" size="1.27" layer="25" ratio="10"/>
+<attribute name="VALUE" x="5.08" y="57.785" size="1.27" layer="27"/>
+</element>
+<element name="PWR_T" library="pinhead" library_urn="urn:adsk.eagle:library:325" package="2X03" package3d_urn="urn:adsk.eagle:package:22462/2" value="" x="46.99" y="29.21" smashed="yes">
+<attribute name="NAME" x="43.18" y="32.385" size="1.27" layer="25" ratio="10"/>
+<attribute name="VALUE" x="43.18" y="24.765" size="1.27" layer="27"/>
+</element>
 <element name="C13" library="resistor" library_urn="urn:adsk.eagle:library:348" package="C050-024X044" package3d_urn="urn:adsk.eagle:package:26162/1" value="100n" x="40.64" y="29.21" smashed="yes" rot="R270">
 <attribute name="VALUE" x="39.2938" y="27.192753125" size="1.27" layer="27" ratio="10" rot="R90"/>
@@
 </signal>
 </signals>
+<mfgpreviewcolors>
+<mfgpreviewcolor name="soldermaskcolor" color="0xC8008000"/>
+<mfgpreviewcolor name="silkscreencolor" color="0xFFFEFEFE"/>
+<mfgpreviewcolor name="backgroundcolor" color="0xFF282828"/>
+<mfgpreviewcolor name="coppercolor" color="0xFFFFBF00"/>
+<mfgpreviewcolor name="substratecolor" color="0xFF786E46"/>
+</mfgpreviewcolors>
 </board>
 </drawing>
