File: Dual LPF/Dual LPF V1.2 Bottom.sch (EAGLE design)
At the start: 48 parts, among them IC2 TL074, IC3 V2164, IC4 TL074

Commit message: Add files via upload
Parts:
- FILM_C1, FILM_C2, FILM_C3, FILM_C4: value 470nF -> 1uF
- R20, R21, R23, R27, R32, R33, R35, R39: value 33k -> 30k
